Commit message: task A.003 done

File: nuturtle_description/urdf/diff_drive.urdf.xacro (robot description, xacro)
@@ -1,9 +1,15 @@
 <?xml version="1.0" ?>
 <robot name="diff_ddrive" xmlns:xacro="https://www.ros.org/wiki/xacro" >
+<xacro:property name="props" value= "${load_yaml('$(find nuturtle_description)/config/diff_params.yaml')}"/>
+<xacro:property name="Wheel_width" value="${props['wheel_width']}" />
+<xacro:property name="wheel_radius" value="${props['wheel_radius']}" />
+<xacro:property name="wheel_base" value="${props['wheel_base']}" />
+<xacro:property name="chassis_length" value="${props['chassis_length']}" />
+<xacro:property name="chassis_thinkness" value="${props['chassis_thinkness']}" />
   <link name="base_link" >
     <visual>
-      <origin rpy="0 0 0" xyz="0 0 0"/>
+      <origin rpy="0 0 0" xyz="0 0 ${wheel_radius}"/>
       <geometry>
-          <box size="0.5 0.3 0.07"/>
+          <box size="${chassis_length} ${wheel_base+Wheel_width} ${chassis_thinkness}"/>
        </geometry>
        <material name="green_mat">
@@ -14,7 +20,7 @@
   <link name="link_right_wheel">
     <visual name="link_right_wheel_visual">
-      <origin rpy="0 1.5707 1.5707" xyz="0 0 0"/>
+      <origin rpy="0 1.5707 1.5707" xyz="0 ${(wheel_base+Wheel_width)/2} ${wheel_radius}"/>
       <geometry>
-        <cylinder length="0.04" radius="0.1"/>
+        <cylinder length="${Wheel_width}" radius="${wheel_radius}"/>
       </geometry>
       <material name="red_mat">
@@ -23,6 +29,6 @@
     </visual>
   </link>
-  <joint name="joint_right_wheel" type="continuous">
-    <origin rpy="0 0 0" xyz="-0.05 0.15 0"/>
+  <joint name="right_wheel_axle" type="continuous">
+    <origin rpy="0 0 0" xyz="0 0 0"/>
     <child link="link_right_wheel"/>
     <parent link="base_link"/>
@@ -33,7 +39,7 @@
   <link name="link_left_wheel">
     <visual name="link_left_wheel_visual">
-      <origin rpy="0 1.5707 1.5707" xyz="0 0 0"/>
+      <origin rpy="0 1.5707 1.5707" xyz="0 ${-(wheel_base+Wheel_width)/2} ${wheel_radius}"/>
       <geometry>
-        <cylinder length="0.04" radius="0.1"/>
+        <cylinder length="${Wheel_width}" radius="${wheel_radius}"/>
       </geometry>
       <material name="red_mat">
@@ -42,6 +48,6 @@
     </visual>
   </link>
-  <joint name="joint_left_wheel" type="continuous">
-    <origin rpy="0 0 0" xyz="0.1 -0.15 0"/>
+  <joint name="left_wheel_axle" type="continuous">
+    <origin rpy="0 0 0" xyz="0 0 0"/>
     <child link="link_left_wheel"/>
     <parent link="base_link"/>
@@ -53,12 +59,12 @@
     <origin rpy=" 0 0 0" xyz="-0.2 0 0.05"/>
     <geometry>
-      <sphere radius="${caster_r}"/>
+      <sphere radius="0.01"/>
     </geometry>
   </visual>
   <link name="link_caster">
     <visual name="caster_visual">
-      <origin rpy="0 0 0" xyz="0 0 0"/>
+      <origin rpy="0 0 0" xyz="${chassis_length/2-wheel_radius/2+chassis_thinkness/4} 0 ${wheel_radius/2-chassis_thinkness/4}"/>
       <geometry>
-        <sphere radius="0.05"/>
+        <sphere radius="${wheel_radius/2-chassis_thinkness/4}"/>
       </geometry>
       <material name="blue_mat">
@@ -68,5 +74,5 @@
   </link>
   <joint name="joint_caster" type="fixed">
-    <origin rpy="0 0 0" xyz="0.1 -0.15 0"/>
+    <origin rpy="0 0 0" xyz="0 0 0"/>
     <child link="link_caster"/>
     <parent link="base_link"/>

Commit message: fixed joint-state-publisher control problem on xacro file, and done with A.002 and A.003

File: nuturtle_description/urdf/diff_drive.urdf.xacro (robot description, xacro)
@@ -20,5 +20,5 @@
   <link name="link_right_wheel">
     <visual name="link_right_wheel_visual">
-      <origin rpy="0 1.5707 1.5707" xyz="0 ${(wheel_base+Wheel_width)/2} ${wheel_radius}"/>
+      <origin rpy="0 1.5707 1.5707" xyz="0 0 0"/>
       <geometry>
         <cylinder length="${Wheel_width}" radius="${wheel_radius}"/>
@@ -30,5 +30,5 @@
   </link>
   <joint name="right_wheel_axle" type="continuous">
-    <origin rpy="0 0 0" xyz="0 0 0"/>
+    <origin rpy="0 0 0" xyz="0 ${(wheel_base+Wheel_width)/2} ${wheel_radius}"/>
     <child link="link_right_wheel"/>
     <parent link="base_link"/>
@@ -39,5 +39,5 @@
   <link name="link_left_wheel">
     <visual name="link_left_wheel_visual">
-      <origin rpy="0 1.5707 1.5707" xyz="0 ${-(wheel_base+Wheel_width)/2} ${wheel_radius}"/>
+      <origin rpy="0 1.5707 1.5707" xyz="0 0 0"/>
       <geometry>
         <cylinder length="${Wheel_width}" radius="${wheel_radius}"/>
@@ -49,5 +49,5 @@
   </link>
   <joint name="left_wheel_axle" type="continuous">
-    <origin rpy="0 0 0" xyz="0 0 0"/>
+    <origin rpy="0 0 0" xyz="0 ${-(wheel_base+Wheel_width)/2} ${wheel_radius}"/>
     <child link="link_left_wheel"/>
     <parent link="base_link"/>

Commit message: start Task B, done B.000

File: nuturtle_description/urdf/diff_drive.urdf.xacro (robot description, xacro)
@@ -56,10 +56,4 @@
     <joint_properties damping="1.0" friction="1.0"/>
   </joint>
-  <visual name="caster_bottom_visual">
-    <origin rpy=" 0 0 0" xyz="-0.2 0 0.05"/>
-    <geometry>
-      <sphere radius="0.01"/>
-    </geometry>
-  </visual>
   <link name="link_caster">
     <visual name="caster_visual">

Commit message: tf works

File: nuturtle_description/urdf/diff_drive.urdf.xacro (robot description, xacro)
@@ -29,5 +29,5 @@
     </visual>
   </link>
-  <joint name="right_wheel_axle" type="continuous">
+  <joint name="odometer/right_wheel_joint" type="continuous">
     <origin rpy="0 0 0" xyz="0 ${(wheel_base+Wheel_width)/2} ${wheel_radius}"/>
     <child link="link_right_wheel"/>
@@ -48,5 +48,5 @@
     </visual>
   </link>
-  <joint name="left_wheel_axle" type="continuous">
+  <joint name="odometer/left_wheel_joint" type="continuous">
     <origin rpy="0 0 0" xyz="0 ${-(wheel_base+Wheel_width)/2} ${wheel_radius}"/>
     <child link="link_left_wheel"/>

Commit message: robot parameter update on urdf

File: nuturtle_description/urdf/diff_drive.urdf.xacro (robot description, xacro)
@@ -7,7 +7,15 @@
 <xacro:property name="chassis_length" value="${props['chassis_length']}" />
 <xacro:property name="chassis_thinkness" value="${props['chassis_thinkness']}" />
+<xacro:property name="wheel_axel_offset" value="${props['wheel_axel_offset']}" />
   <link name="base_link" >
+    <pose>0 0 ${chassis_thinkness/2 + wheel_radius-0.02} 0 0 0</pose>
+<!--
+    <inertial>
+      <mass value="0.94"/>
+      <origin rpy="0 0 0" xyz="0 0 ${chassis_thinkness/2 + wheel_radius-0.02}"/>
+      <inertia ixx="0.0395416666667" ixy="0" ixz="0" iyy="0.106208333333" iyz="0" izz="0.106208333333"/>
+    </inertial> -->
     <visual>
-      <origin rpy="0 0 0" xyz="0 0 ${wheel_radius}"/>
+      <origin rpy="0 0 0" xyz="0 0 ${chassis_thinkness/2 + wheel_radius-0.02}"/>
       <geometry>
           <box size="${chassis_length} ${wheel_base+Wheel_width} ${chassis_thinkness}"/>
@@ -20,5 +28,5 @@
   <link name="link_right_wheel">
     <visual name="link_right_wheel_visual">
-      <origin rpy="0 1.5707 1.5707" xyz="0 0 0"/>
+      <origin rpy="0 1.5707 1.5707" xyz="${wheel_radius} 0 0"/>
       <geometry>
         <cylinder length="${Wheel_width}" radius="${wheel_radius}"/>
@@ -39,5 +47,5 @@
   <link name="link_left_wheel">
     <visual name="link_left_wheel_visual">
-      <origin rpy="0 1.5707 1.5707" xyz="0 0 0"/>
+      <origin rpy="0 1.5707 1.5707" xyz="${wheel_radius} 0 0"/>
       <geometry>
         <cylinder length="${Wheel_width}" radius="${wheel_radius}"/>
@@ -58,10 +66,10 @@
   <link name="link_caster">
     <visual name="caster_visual">
-      <origin rpy="0 0 0" xyz="${chassis_length/2-wheel_radius/2+chassis_thinkness/4} 0 ${wheel_radius/2-chassis_thinkness/4}"/>
+      <origin rpy="0 0 0" xyz="${-chassis_length/2 + (wheel_radius/2-wheel_axel_offset/2)} 0 ${wheel_radius/2-wheel_axel_offset/2}"/>
       <geometry>
-        <sphere radius="${wheel_radius/2-chassis_thinkness/4}"/>
+        <sphere radius="${wheel_radius/2-wheel_axel_offset/2}"/>
       </geometry>
-      <material name="blue_mat">
-        <color rgba="0.203125 0.23828125 0.28515625 1.0"/>
+      <material name="red_mat">
+        <color rgba="1 0 0 0.5"/>
       </material>
     </visual>

Commit message: fix wheel joint on urdf

File: nuturtle_description/urdf/diff_drive.urdf.xacro (robot description, xacro)
@@ -9,13 +9,12 @@
 <xacro:property name="wheel_axel_offset" value="${props['wheel_axel_offset']}" />
   <link name="base_link" >
-    <pose>0 0 ${chassis_thinkness/2 + wheel_radius-0.02} 0 0 0</pose>
-<!--
+    <pose>0 0 ${chassis_thinkness/2 + wheel_radius-wheel_axel_offset} 0 0 0</pose>
     <inertial>
       <mass value="0.94"/>
-      <origin rpy="0 0 0" xyz="0 0 ${chassis_thinkness/2 + wheel_radius-0.02}"/>
+      <origin rpy="0 0 0" xyz="0 0 ${chassis_thinkness/2 + wheel_radius-wheel_axel_offset}"/>
       <inertia ixx="0.0395416666667" ixy="0" ixz="0" iyy="0.106208333333" iyz="0" izz="0.106208333333"/>
-    </inertial> -->
+    </inertial>
     <visual>
-      <origin rpy="0 0 0" xyz="0 0 ${chassis_thinkness/2 + wheel_radius-0.02}"/>
+      <origin rpy="0 0 0" xyz="0 0 ${chassis_thinkness/2 + wheel_radius-wheel_axel_offset}"/>
       <geometry>
           <box size="${chassis_length} ${wheel_base+Wheel_width} ${chassis_thinkness}"/>
@@ -28,5 +27,5 @@
   <link name="link_right_wheel">
     <visual name="link_right_wheel_visual">
-      <origin rpy="0 1.5707 1.5707" xyz="${wheel_radius} 0 0"/>
+      <origin rpy="0 1.5707 1.5707" xyz="0 0 0"/>
       <geometry>
         <cylinder length="${Wheel_width}" radius="${wheel_radius}"/>
@@ -38,5 +37,5 @@
   </link>
   <joint name="odometer/right_wheel_joint" type="continuous">
-    <origin rpy="0 0 0" xyz="0 ${(wheel_base+Wheel_width)/2} ${wheel_radius}"/>
+    <origin rpy="0 0 0" xyz="${wheel_radius} ${(wheel_base+Wheel_width)/2} ${wheel_radius}"/>
     <child link="link_right_wheel"/>
     <parent link="base_link"/>
@@ -47,5 +46,5 @@
   <link name="link_left_wheel">
     <visual name="link_left_wheel_visual">
-      <origin rpy="0 1.5707 1.5707" xyz="${wheel_radius} 0 0"/>
+      <origin rpy="0 1.5707 1.5707" xyz="0 0 0"/>
       <geometry>
         <cylinder length="${Wheel_width}" radius="${wheel_radius}"/>
@@ -57,5 +56,5 @@
   </link>
   <joint name="odometer/left_wheel_joint" type="continuous">
-    <origin rpy="0 0 0" xyz="0 ${-(wheel_base+Wheel_width)/2} ${wheel_radius}"/>
+    <origin rpy="0 0 0" xyz="${wheel_radius} ${-(wheel_base+Wheel_width)/2} ${wheel_radius}"/>
     <child link="link_left_wheel"/>
     <parent link="base_link"/>

Commit message: task A004 done

File: nuturtle_description/urdf/diff_drive.urdf.xacro (robot description, xacro)
@@ -8,4 +8,5 @@
 <xacro:property name="chassis_thinkness" value="${props['chassis_thinkness']}" />
 <xacro:property name="wheel_axel_offset" value="${props['wheel_axel_offset']}" />
+<xacro:include filename="$(find nuturtle_description)/urdf/macro.xacro" />
   <link name="base_link" >
     <pose>0 0 ${chassis_thinkness/2 + wheel_radius-wheel_axel_offset} 0 0 0</pose>
@@ -13,6 +14,11 @@
       <mass value="0.94"/>
       <origin rpy="0 0 0" xyz="0 0 ${chassis_thinkness/2 + wheel_radius-wheel_axel_offset}"/>
-      <inertia ixx="0.0395416666667" ixy="0" ixz="0" iyy="0.106208333333" iyz="0" izz="0.106208333333"/>
+      <inertia ixx="${0.94*((wheel_base+Wheel_width)*(wheel_base+Wheel_width)+chassis_thinkness*chassis_thinkness)/12.0}" ixy="0" ixz="0" iyy="${0.94*(chassis_length*chassis_length+chassis_thinkness*chassis_thinkness)/12.0}" iyz="0" izz="${0.94*((wheel_base+Wheel_width)*(wheel_base+Wheel_width)+chassis_length*chassis_length)/12.0}"/>
     </inertial>
+    <collision name="collision_chassis">
+      <geometry>
+        <box size="${chassis_length} ${wheel_base+Wheel_width} ${chassis_thinkness}"/>
+      </geometry>
+    </collision>
     <visual>
       <origin rpy="0 0 0" xyz="0 0 ${chassis_thinkness/2 + wheel_radius-wheel_axel_offset}"/>
@@ -20,10 +26,45 @@
           <box size="${chassis_length} ${wheel_base+Wheel_width} ${chassis_thinkness}"/>
        </geometry>
-       <material name="green_mat">
-           <color rgba="0 1 0 1" />
+       <material name="black_mat">
+           <color rgba="0.203125 0.23828125 0.28515625 1.0"/>
        </material>
      </visual>
+     <!-- caster front -->
+     <collision name="caster_top_collision">
+       <origin rpy="0 0 0" xyz="${-chassis_length/2 + (wheel_radius/2-wheel_axel_offset/2)} 0 ${wheel_radius/2-wheel_axel_offset/2}"/>
+       <geometry>
+         <sphere radius="${wheel_radius/2-wheel_axel_offset/2}"/>
+       </geometry>
+       <surface>
+         <friction>
+           <ode>
+             <mu>0</mu>
+             <mu2>0</mu2>
+             <slip1>1.0</slip1>
+             <slip2>1.0</slip2>
+           </ode>
+         </friction>
+       </surface>
+     </collision>
+     <visual name="caster_top_visual">
+      <origin rpy="0 0 0" xyz="${-chassis_length/2 + (wheel_radius/2-wheel_axel_offset/2)} 0 ${wheel_radius/2-wheel_axel_offset/2}"/>
+       <geometry>
+         <sphere radius="${wheel_radius/2-wheel_axel_offset/2}"/>
+         <!-- </material> -->
+       </geometry>
+     </visual>
   </link>
-  <link name="link_right_wheel">
+  <!-- <link name="link_right_wheel">
+    <inertial>
+      <mass value="0.03"/>
+      <origin rpy="0 1.5707 1.5707" xyz="0 0 0"/>
+      <inertia ixx="${0.03*(3*wheel_radius*wheel_radius+Wheel_width*Wheel_width)/12.0}" ixy="0" ixz="0" iyy="${0.03*(3*wheel_radius*wheel_radius+Wheel_width*Wheel_width)/12.0}" iyz="0" izz="${0.03*wheel_radius*wheel_radius/2.0}"/>
+    </inertial>
+    <collision name="link_right_collision">
+      <origin rpy="0 1.5707 1.5707" xyz="0 0 0"/>
+      <geometry>
+        <cylinder length="${Wheel_width}" radius="${wheel_radius}"/>
+      </geometry>
+    </collision>
     <visual name="link_right_wheel_visual">
       <origin rpy="0 1.5707 1.5707" xyz="0 0 0"/>
@@ -62,19 +103,15 @@
     <limit effort="10000" velocity="1000"/>
     <joint_properties damping="1.0" friction="1.0"/>
-  </joint>
-  <link name="link_caster">
-    <visual name="caster_visual">
-      <origin rpy="0 0 0" xyz="${-chassis_length/2 + (wheel_radius/2-wheel_axel_offset/2)} 0 ${wheel_radius/2-wheel_axel_offset/2}"/>
-      <geometry>
-        <sphere radius="${wheel_radius/2-wheel_axel_offset/2}"/>
-      </geometry>
-      <material name="red_mat">
-        <color rgba="1 0 0 0.5"/>
-      </material>
-    </visual>
+  </joint> -->
+  <xacro:link_wheel name="link_right_wheel" />
+  <xacro:joint_wheel name="odometer/right_wheel_joint"  child="link_right_wheel"  origin_xyz="${wheel_radius} ${(wheel_base+Wheel_width)/2} ${wheel_radius}"  />
+  <xacro:link_wheel name="link_left_wheel" />
+  <xacro:joint_wheel name="odometer/left_wheel_joint"   child="link_left_wheel"   origin_xyz="${wheel_radius} ${-(wheel_base+Wheel_width)/2} ${wheel_radius}"  />
+  <link name="base_scan">
+      <origin rpy="0 0 1.5707" xyz="0 0 ${wheel_radius-0.02+chassis_thinkness}"/>
   </link>
   <joint name="joint_caster" type="fixed">
-    <origin rpy="0 0 0" xyz="0 0 0"/>
-    <child link="link_caster"/>
+    <origin rpy="0 0 0" xyz="0 0 ${wheel_radius-0.02+chassis_thinkness}"/>
+    <child link="base_scan"/>
     <parent link="base_link"/>
   </joint>

Commit message: G001 and G002 done

File: nuturtle_description/urdf/diff_drive.urdf.xacro (robot description, xacro)
@@ -9,5 +9,11 @@
 <xacro:property name="wheel_axel_offset" value="${props['wheel_axel_offset']}" />
 <xacro:include filename="$(find nuturtle_description)/urdf/macro.xacro" />
-  <link name="base_link" >
+<xacro:include filename="$(find nuturtle_gazebo)/urdf/diff_drive.gazebo" />
+<xacro:include filename="$(find nuturtle_gazebo)/urdf/material.urdf.xacro" />
+<xacro:arg name="mode" default="0" />
+  <link name="base_link">
+      <origin rpy="0 0 0" xyz="0 0 0"/>
+  </link>
+  <link name="base_body" >
     <pose>0 0 ${chassis_thinkness/2 + wheel_radius-wheel_axel_offset} 0 0 0</pose>
     <inertial>
@@ -17,4 +23,5 @@
     </inertial>
     <collision name="collision_chassis">
+      <origin rpy="0 0 0" xyz="0 0 ${chassis_thinkness/2 + wheel_radius-wheel_axel_offset}"/>
       <geometry>
         <box size="${chassis_length} ${wheel_base+Wheel_width} ${chassis_thinkness}"/>
@@ -26,7 +33,7 @@
           <box size="${chassis_length} ${wheel_base+Wheel_width} ${chassis_thinkness}"/>
        </geometry>
-       <material name="black_mat">
+       <!-- <material name="black_mat">
            <color rgba="0.203125 0.23828125 0.28515625 1.0"/>
-       </material>
+       </material> -->
      </visual>
      <!-- caster front -->
@@ -39,8 +46,10 @@
          <friction>
            <ode>
-             <mu>0</mu>
-             <mu2>0</mu2>
-             <slip1>1.0</slip1>
-             <slip2>1.0</slip2>
+             <mu>0.0</mu>
+             <mu2>0.0</mu2>
+             <minDepth>0.001</minDepth>
+             <maxVel>1.0</maxVel>
+             <kp>1000000</kp>
+             <kd>100</kd>
            </ode>
          </friction>
@@ -51,61 +60,12 @@
        <geometry>
          <sphere radius="${wheel_radius/2-wheel_axel_offset/2}"/>
-         <!-- </material> -->
        </geometry>
      </visual>
   </link>
-  <!-- <link name="link_right_wheel">
-    <inertial>
-      <mass value="0.03"/>
-      <origin rpy="0 1.5707 1.5707" xyz="0 0 0"/>
-      <inertia ixx="${0.03*(3*wheel_radius*wheel_radius+Wheel_width*Wheel_width)/12.0}" ixy="0" ixz="0" iyy="${0.03*(3*wheel_radius*wheel_radius+Wheel_width*Wheel_width)/12.0}" iyz="0" izz="${0.03*wheel_radius*wheel_radius/2.0}"/>
-    </inertial>
-    <collision name="link_right_collision">
-      <origin rpy="0 1.5707 1.5707" xyz="0 0 0"/>
-      <geometry>
-        <cylinder length="${Wheel_width}" radius="${wheel_radius}"/>
-      </geometry>
-    </collision>
-    <visual name="link_right_wheel_visual">
-      <origin rpy="0 1.5707 1.5707" xyz="0 0 0"/>
-      <geometry>
-        <cylinder length="${Wheel_width}" radius="${wheel_radius}"/>
-      </geometry>
-      <material name="red_mat">
-          <color rgba="1 0 0 0.5" />
-      </material>
-    </visual>
-  </link>
-  <joint name="odometer/right_wheel_joint" type="continuous">
-    <origin rpy="0 0 0" xyz="${wheel_radius} ${(wheel_base+Wheel_width)/2} ${wheel_radius}"/>
-    <child link="link_right_wheel"/>
-    <parent link="base_link"/>
-    <axis rpy="0 0 0" xyz="0 1 0"/>
-    <limit effort="10000" velocity="1000"/>
-    <joint_properties damping="1.0" friction="1.0"/>
-  </joint>
-  <link name="link_left_wheel">
-    <visual name="link_left_wheel_visual">
-      <origin rpy="0 1.5707 1.5707" xyz="0 0 0"/>
-      <geometry>
-        <cylinder length="${Wheel_width}" radius="${wheel_radius}"/>
-      </geometry>
-      <material name="red_mat">
-          <color rgba="1 0 0 0.5" />
-      </material>
-    </visual>
-  </link>
-  <joint name="odometer/left_wheel_joint" type="continuous">
-    <origin rpy="0 0 0" xyz="${wheel_radius} ${-(wheel_base+Wheel_width)/2} ${wheel_radius}"/>
-    <child link="link_left_wheel"/>
-    <parent link="base_link"/>
-    <axis rpy="0 0 0" xyz="0 1 0"/>
-    <limit effort="10000" velocity="1000"/>
-    <joint_properties damping="1.0" friction="1.0"/>
-  </joint> -->
   <xacro:link_wheel name="link_right_wheel" />
   <xacro:joint_wheel name="odometer/right_wheel_joint"  child="link_right_wheel"  origin_xyz="${wheel_radius} ${(wheel_base+Wheel_width)/2} ${wheel_radius}"  />
   <xacro:link_wheel name="link_left_wheel" />
   <xacro:joint_wheel name="odometer/left_wheel_joint"   child="link_left_wheel"   origin_xyz="${wheel_radius} ${-(wheel_base+Wheel_width)/2} ${wheel_radius}"  />
+  <!-- <xacro:robot_dd mode="$(arg mode)" /> -->
   <link name="base_scan">
       <origin rpy="0 0 1.5707" xyz="0 0 ${wheel_radius-0.02+chassis_thinkness}"/>
@@ -114,5 +74,11 @@
     <origin rpy="0 0 0" xyz="0 0 ${wheel_radius-0.02+chassis_thinkness}"/>
     <child link="base_scan"/>
+    <parent link="base_body"/>
+  </joint>
+  <joint name="base_link_base_body_joint" type="fixed">
+    <origin rpy="0 0 0" xyz="0 0 0"/>
+    <child link="base_body"/>
     <parent link="base_link"/>
   </joint>
+  <xacro:robot_dd mode="$(arg mode)" />
 </robot>

File: nuturtle_description/urdf/macro.xacro (robot description, xacro)
@@ -4,7 +4,7 @@
         <link name="${name}">
             <inertial>
-              <mass value="0.1"/>
+              <mass value="0.03"/>
               <origin rpy="0 1.5707 1.5707" xyz="0 0 0"/>
-              <inertia ixx="0.000526666666667" ixy="0" ixz="0" iyy="0.000526666666667" iyz="0" izz="0.001"/>
+              <inertia ixx="${0.03*(3*wheel_radius*wheel_radius+Wheel_width*Wheel_width)/12.0}" ixy="0" ixz="0" iyy="${0.03*(3*wheel_radius*wheel_radius+Wheel_width*Wheel_width)/12.0}" iyz="0" izz="${0.03*wheel_radius*wheel_radius/2.0}"/>
             </inertial>
             <collision name="${name}_collision">
@@ -13,4 +13,17 @@
                 <cylinder length="${Wheel_width}" radius="${wheel_radius}"/>
               </geometry>
+              <surface>
+                <friction>
+                  <ode>
+                    <mu1>0.3</mu1>
+                    <mu2>0.3</mu2>
+                    <minDepth>0.001</minDepth>
+                    <fdir1>1 0 0 </fdir1>
+                    <maxVel>0.1</maxVel>
+                    <kp>500000</kp>
+                    <kd>10</kd>
+                  </ode>
+                </friction>
+              </surface>
             </collision>
             <visual name="${name}_visual">
@@ -26,5 +39,5 @@
         <origin rpy="0 0 0" xyz="${origin_xyz}"/>
         <child link="${child}"/>
-        <parent link="base_link"/>
+        <parent link="base_body"/>
         <axis rpy="0 0 0" xyz="0 1 0"/>
         <limit effort="10000" velocity="1000"/>
