Commit message: done part G

File: nuturtle_description/urdf/diff_drive.urdf.xacro (robot description, xacro)
@@ -22,5 +22,5 @@
       <inertia ixx="${0.94*((wheel_base+Wheel_width)*(wheel_base+Wheel_width)+chassis_thinkness*chassis_thinkness)/12.0}" ixy="0" ixz="0" iyy="${0.94*(chassis_length*chassis_length+chassis_thinkness*chassis_thinkness)/12.0}" iyz="0" izz="${0.94*((wheel_base+Wheel_width)*(wheel_base+Wheel_width)+chassis_length*chassis_length)/12.0}"/>
     </inertial>
-    <collision name="collision_chassis">
+    <collision>
       <origin rpy="0 0 0" xyz="0 0 ${chassis_thinkness/2 + wheel_radius-wheel_axel_offset}"/>
       <geometry>
@@ -33,8 +33,7 @@
           <box size="${chassis_length} ${wheel_base+Wheel_width} ${chassis_thinkness}"/>
        </geometry>
-       <!-- <material name="black_mat">
-           <color rgba="0.203125 0.23828125 0.28515625 1.0"/>
-       </material> -->
      </visual>
+  </link>
+   <link name="ball_caster">
      <!-- caster front -->
      <collision name="caster_top_collision">
@@ -43,18 +42,6 @@
          <sphere radius="${wheel_radius/2-wheel_axel_offset/2}"/>
        </geometry>
-       <surface>
-         <friction>
-           <ode>
-             <mu>0.0</mu>
-             <mu2>0.0</mu2>
-             <minDepth>0.001</minDepth>
-             <maxVel>1.0</maxVel>
-             <kp>1000000</kp>
-             <kd>100</kd>
-           </ode>
-         </friction>
-       </surface>
      </collision>
-     <visual name="caster_top_visual">
+     <visual>
       <origin rpy="0 0 0" xyz="${-chassis_length/2 + (wheel_radius/2-wheel_axel_offset/2)} 0 ${wheel_radius/2-wheel_axel_offset/2}"/>
        <geometry>
@@ -81,4 +68,9 @@
     <parent link="base_link"/>
   </joint>
+  <joint name="caster_chassis" type="fixed">
+    <parent link="base_body"/>
+    <child link="ball_caster"/>
+    <origin rpy="0 0 0" xyz="0 0 0"/>
+  </joint>
   <xacro:robot_dd mode="$(arg mode)" />
 </robot>

File: nuturtle_description/urdf/macro.xacro (robot description, xacro)
@@ -13,9 +13,9 @@
                 <cylinder length="${Wheel_width}" radius="${wheel_radius}"/>
               </geometry>
-              <surface>
+              <!-- <surface>
                 <friction>
                   <ode>
-                    <mu1>0.3</mu1>
-                    <mu2>0.3</mu2>
+                    <mu1>0</mu1>
+                    <mu2>0</mu2>
                     <minDepth>0.001</minDepth>
                     <fdir1>1 0 0 </fdir1>
@@ -25,5 +25,5 @@
                   </ode>
                 </friction>
-              </surface>
+              </surface> -->
             </collision>
             <visual name="${name}_visual">

Commit message: reformat nu_description package

File: nuturtle_description/urdf/diff_drive.urdf.xacro (robot description, xacro)
@@ -1,4 +1,4 @@
 <?xml version="1.0" ?>
-<robot name="diff_ddrive" xmlns:xacro="https://www.ros.org/wiki/xacro" >
+<robot name="diff_drive" xmlns:xacro="https://www.ros.org/wiki/xacro" >
 <xacro:property name="props" value= "${load_yaml('$(find nuturtle_description)/config/diff_params.yaml')}"/>
 <xacro:property name="Wheel_width" value="${props['wheel_width']}" />
@@ -6,9 +6,9 @@
 <xacro:property name="wheel_base" value="${props['wheel_base']}" />
 <xacro:property name="chassis_length" value="${props['chassis_length']}" />
-<xacro:property name="chassis_thinkness" value="${props['chassis_thinkness']}" />
+<xacro:property name="chassis_thickness" value="${props['chassis_thickness']}" />
 <xacro:property name="wheel_axel_offset" value="${props['wheel_axel_offset']}" />
 <xacro:include filename="$(find nuturtle_description)/urdf/macro.xacro" />
-<xacro:include filename="$(find nuturtle_gazebo)/urdf/diff_drive.gazebo" />
-<xacro:include filename="$(find nuturtle_gazebo)/urdf/material.urdf.xacro" />
+<!-- <xacro:include filename="$(find nuturtle_gazebo)/urdf/diff_drive.gazebo" /> -->
+<!-- <xacro:include filename="$(find nuturtle_gazebo)/urdf/material.urdf.xacro" /> -->
 <xacro:arg name="mode" default="0" />
   <link name="base_link">
@@ -16,51 +16,53 @@
   </link>
   <link name="base_body" >
-    <pose>0 0 ${chassis_thinkness/2 + wheel_radius-wheel_axel_offset} 0 0 0</pose>
+    <!-- <pose>0 0 ${chassis_thickness/2 + wheel_radius-wheel_axel_offset} 0 0 0</pose> -->
+<!--
     <inertial>
       <mass value="0.94"/>
-      <origin rpy="0 0 0" xyz="0 0 ${chassis_thinkness/2 + wheel_radius-wheel_axel_offset}"/>
-      <inertia ixx="${0.94*((wheel_base+Wheel_width)*(wheel_base+Wheel_width)+chassis_thinkness*chassis_thinkness)/12.0}" ixy="0" ixz="0" iyy="${0.94*(chassis_length*chassis_length+chassis_thinkness*chassis_thinkness)/12.0}" iyz="0" izz="${0.94*((wheel_base+Wheel_width)*(wheel_base+Wheel_width)+chassis_length*chassis_length)/12.0}"/>
+      <origin rpy="0 0 0" xyz="0 0 ${chassis_thickness/2 + wheel_radius-wheel_axel_offset}"/>
+      <inertia ixx="${0.94*((wheel_base+Wheel_width)*(wheel_base+Wheel_width)+chassis_thickness*chassis_thickness)/12.0}" ixy="0" ixz="0" iyy="${0.94*(chassis_length*chassis_length+chassis_thickness*chassis_thickness)/12.0}" iyz="0" izz="${0.94*((wheel_base+Wheel_width)*(wheel_base+Wheel_width)+chassis_length*chassis_length)/12.0}"/>
     </inertial>
     <collision>
-      <origin rpy="0 0 0" xyz="0 0 ${chassis_thinkness/2 + wheel_radius-wheel_axel_offset}"/>
+      <origin rpy="0 0 0" xyz="0 0 ${chassis_thickness/2 + wheel_radius-wheel_axel_offset}"/>
       <geometry>
-        <box size="${chassis_length} ${wheel_base+Wheel_width} ${chassis_thinkness}"/>
+        <box size="${chassis_length} ${wheel_base-Wheel_width} ${chassis_thickness}"/>
       </geometry>
-    </collision>
+    </collision> -->
     <visual>
-      <origin rpy="0 0 0" xyz="0 0 ${chassis_thinkness/2 + wheel_radius-wheel_axel_offset}"/>
+      <origin rpy="0 0 0" xyz="0 0 ${chassis_thickness/2 + wheel_radius-wheel_axel_offset}"/>
       <geometry>
-          <box size="${chassis_length} ${wheel_base+Wheel_width} ${chassis_thinkness}"/>
+          <box size="${chassis_length} ${wheel_base-Wheel_width} ${chassis_thickness}"/>
        </geometry>
      </visual>
   </link>
    <link name="ball_caster">
-     <!-- caster front -->
-     <collision name="caster_top_collision">
-       <origin rpy="0 0 0" xyz="${-chassis_length/2 + (wheel_radius/2-wheel_axel_offset/2)} 0 ${wheel_radius/2-wheel_axel_offset/2}"/>
+     <!-- <collision name="caster_top_collision">
+       <origin rpy="0 0 0" xyz="${chassis_length/2 - (wheel_radius/2-wheel_axel_offset/2)} 0 ${wheel_radius/2-wheel_axel_offset/2}"/>
        <geometry>
          <sphere radius="${wheel_radius/2-wheel_axel_offset/2}"/>
        </geometry>
-     </collision>
+     </collision> -->
      <visual>
-      <origin rpy="0 0 0" xyz="${-chassis_length/2 + (wheel_radius/2-wheel_axel_offset/2)} 0 ${wheel_radius/2-wheel_axel_offset/2}"/>
+      <origin rpy="0 0 0" xyz="${chassis_length/2 - (wheel_radius/2-wheel_axel_offset/2)} 0 ${wheel_radius/2-wheel_axel_offset/2}"/>
        <geometry>
          <sphere radius="${wheel_radius/2-wheel_axel_offset/2}"/>
        </geometry>
+       <material name="blue">
+                <color rgba="0 0 1 1" />
+       </material>
      </visual>
   </link>
   <xacro:link_wheel name="link_right_wheel" />
-  <xacro:joint_wheel name="odometer/right_wheel_joint"  child="link_right_wheel"  origin_xyz="${wheel_radius} ${(wheel_base+Wheel_width)/2} ${wheel_radius}"  />
+  <xacro:joint_wheel name="odometer/right_wheel_joint"  child="link_right_wheel"  origin_xyz="${wheel_radius} ${(wheel_base)/2} ${wheel_radius}"  />
   <xacro:link_wheel name="link_left_wheel" />
-  <xacro:joint_wheel name="odometer/left_wheel_joint"   child="link_left_wheel"   origin_xyz="${wheel_radius} ${-(wheel_base+Wheel_width)/2} ${wheel_radius}"  />
-  <!-- <xacro:robot_dd mode="$(arg mode)" /> -->
-  <link name="base_scan">
-      <origin rpy="0 0 1.5707" xyz="0 0 ${wheel_radius-0.02+chassis_thinkness}"/>
-  </link>
-  <joint name="joint_caster" type="fixed">
-    <origin rpy="0 0 0" xyz="0 0 ${wheel_radius-0.02+chassis_thinkness}"/>
+  <xacro:joint_wheel name="odometer/left_wheel_joint"   child="link_left_wheel"   origin_xyz="${wheel_radius} ${-(wheel_base)/2} ${wheel_radius}"  />
+  <!-- <link name="base_scan">
+      <origin rpy="0 0 1.5707" xyz="0 0 ${wheel_radius-0.02+chassis_thickness}"/>
+  </link> -->
+  <!-- <joint name="joint_caster" type="fixed">
+    <origin rpy="0 0 0" xyz="0 0 ${wheel_radius-0.02+chassis_thickness}"/>
     <child link="base_scan"/>
     <parent link="base_body"/>
-  </joint>
+  </joint> -->
   <joint name="base_link_base_body_joint" type="fixed">
     <origin rpy="0 0 0" xyz="0 0 0"/>
@@ -73,4 +75,4 @@
     <origin rpy="0 0 0" xyz="0 0 0"/>
   </joint>
-  <xacro:robot_dd mode="$(arg mode)" />
+  <!-- <xacro:robot_dd mode="$(arg mode)" /> -->
 </robot>

File: nuturtle_description/urdf/macro.xacro (robot description, xacro)
@@ -3,15 +3,15 @@
     <xacro:macro name="link_wheel" params="name">
         <link name="${name}">
-            <inertial>
+            <!-- <inertial>
               <mass value="0.03"/>
-              <origin rpy="0 1.5707 1.5707" xyz="0 0 0"/>
+              <origin rpy="1.5707 0 0" xyz="0 0 0"/>
               <inertia ixx="${0.03*(3*wheel_radius*wheel_radius+Wheel_width*Wheel_width)/12.0}" ixy="0" ixz="0" iyy="${0.03*(3*wheel_radius*wheel_radius+Wheel_width*Wheel_width)/12.0}" iyz="0" izz="${0.03*wheel_radius*wheel_radius/2.0}"/>
             </inertial>
             <collision name="${name}_collision">
-              <origin rpy="0 1.5707 1.5707" xyz="0 0 0"/>
+              <origin rpy="1.5707 0 0" xyz="0 0 0"/>
               <geometry>
                 <cylinder length="${Wheel_width}" radius="${wheel_radius}"/>
               </geometry>
-              <!-- <surface>
+              <surface>
                 <friction>
                   <ode>
@@ -25,11 +25,14 @@
                   </ode>
                 </friction>
-              </surface> -->
-            </collision>
+              </surface>
+            </collision> -->
             <visual name="${name}_visual">
-              <origin rpy="0 1.5707 1.5707" xyz="0 0 0"/>
+              <origin rpy="1.5707 0 0" xyz="0 0 0"/>
               <geometry>
                 <cylinder length="${Wheel_width}" radius="${wheel_radius}"/>
               </geometry>
+              <material name="yellow">
+                <color rgba="1 1 0 1.0" />
+              </material>
             </visual>
         </link>

Commit message: done

File: nuturtle_description/urdf/diff_drive.urdf.xacro (robot description, xacro)
@@ -9,5 +9,5 @@
 <xacro:property name="wheel_axel_offset" value="${props['wheel_axel_offset']}" />
 <xacro:include filename="$(find nuturtle_description)/urdf/macro.xacro" />
-<!-- <xacro:include filename="$(find nuturtle_gazebo)/urdf/diff_drive.gazebo" /> -->
+<xacro:include filename="$(find nuturtle_gazebo)/urdf/diff_drive.gazebo" />
 <!-- <xacro:include filename="$(find nuturtle_gazebo)/urdf/material.urdf.xacro" /> -->
 <xacro:arg name="mode" default="0" />
@@ -16,10 +16,8 @@
   </link>
   <link name="base_body" >
-    <!-- <pose>0 0 ${chassis_thickness/2 + wheel_radius-wheel_axel_offset} 0 0 0</pose> -->
-<!--
     <inertial>
-      <mass value="0.94"/>
+      <mass value="1.0"/>
       <origin rpy="0 0 0" xyz="0 0 ${chassis_thickness/2 + wheel_radius-wheel_axel_offset}"/>
-      <inertia ixx="${0.94*((wheel_base+Wheel_width)*(wheel_base+Wheel_width)+chassis_thickness*chassis_thickness)/12.0}" ixy="0" ixz="0" iyy="${0.94*(chassis_length*chassis_length+chassis_thickness*chassis_thickness)/12.0}" iyz="0" izz="${0.94*((wheel_base+Wheel_width)*(wheel_base+Wheel_width)+chassis_length*chassis_length)/12.0}"/>
+      <inertia ixx="${1.0*((wheel_base-Wheel_width)*(wheel_base-Wheel_width)+chassis_thickness*chassis_thickness)/12.0}" ixy="0" ixz="0" iyy="${1.0*(chassis_length*chassis_length+(wheel_base-Wheel_width)*(wheel_base-Wheel_width))/12.0}" iyz="0" izz="${1.0*(chassis_thickness*chassis_thickness + chassis_length*chassis_length)/12.0}"/>
     </inertial>
     <collision>
@@ -28,5 +26,5 @@
         <box size="${chassis_length} ${wheel_base-Wheel_width} ${chassis_thickness}"/>
       </geometry>
-    </collision> -->
+    </collision>
     <visual>
       <origin rpy="0 0 0" xyz="0 0 ${chassis_thickness/2 + wheel_radius-wheel_axel_offset}"/>
@@ -37,10 +35,10 @@
   </link>
    <link name="ball_caster">
-     <!-- <collision name="caster_top_collision">
+     <collision name="caster_top_collision">
        <origin rpy="0 0 0" xyz="${chassis_length/2 - (wheel_radius/2-wheel_axel_offset/2)} 0 ${wheel_radius/2-wheel_axel_offset/2}"/>
        <geometry>
          <sphere radius="${wheel_radius/2-wheel_axel_offset/2}"/>
        </geometry>
-     </collision> -->
+     </collision>
      <visual>
       <origin rpy="0 0 0" xyz="${chassis_length/2 - (wheel_radius/2-wheel_axel_offset/2)} 0 ${wheel_radius/2-wheel_axel_offset/2}"/>
@@ -57,12 +55,17 @@
   <xacro:link_wheel name="link_left_wheel" />
   <xacro:joint_wheel name="left_wheel_joint"   child="link_left_wheel"   origin_xyz="${wheel_radius} ${-(wheel_base)/2} ${wheel_radius}"  />
-  <!-- <link name="base_scan">
-      <origin rpy="0 0 1.5707" xyz="0 0 ${wheel_radius-0.02+chassis_thickness}"/>
-  </link> -->
-  <!-- <joint name="joint_caster" type="fixed">
-    <origin rpy="0 0 0" xyz="0 0 ${wheel_radius-0.02+chassis_thickness}"/>
+  <!-- add base scan link  -->
+  <link name="base_scan">
+      <visual name="base_scan_visual">
+          <geometry>
+              <cylinder radius="0.01" length="0.01"/>
+          </geometry>
+      </visual>
+  </link>
+  <joint name="joint_caster" type="fixed">
+    <origin rpy="0 0 0" xyz="0 0 ${wheel_radius-wheel_axel_offset+chassis_thickness/2}"/>
     <child link="base_scan"/>
     <parent link="base_body"/>
-  </joint> -->
+  </joint>
   <joint name="base_link_base_body_joint" type="fixed">
     <origin rpy="0 0 0" xyz="0 0 0"/>
